Commit message: Added thrust. Change of axis not working yet.

File: servorobots/quad.urdf (robot description, URDF)
Before this commit: robot physics, 1 links, 0 joints
Links:
- link baseLink: mass .1 -> .6; geometry collision box size=.25 .25 .05; visual mesh filename=/model/quadcopter.obj scale=1 1 1
