Commit message: Almost working robot

File: servorobots/balancer.urdf (robot description, URDF)
Before this commit: robot physics, 3 links, 2 joints
Links:
- link baseLink: mass .6 -> .3; geometry collision box size=0.08 0.1 0.04; visual box size=0.04 0.085 0.11
- link wheel_left: mass .6 -> .01
- link wheel_right: mass .6 -> .01
Joints:
- joint wheel_left_joint: origin xyz=0 0.151 0 rpy=1.5708 0 0 -> xyz=0 0.051 0 rpy=1.5708 0 0
- joint wheel_right_joint: origin xyz=0 -0.151 0 rpy=1.5708 0 0 -> xyz=0 -0.051 0 rpy=1.5708 0 0

Commit message: Progress!

File: servorobots/balancer.urdf (robot description, URDF)
Before this commit: robot physics, 3 links, 2 joints
Links:
- link baseLink: geometry collision box size=0.20 0.1 0.04; visual box size=0.04 0.085 0.11

File: servorobots/balancer_spring.urdf (robot description, URDF)
Before this commit: robot physics, 5 links, 2 joints
Links:
- link baseLink: geometry collision box size=0.015 0.1 0.04; visual box size=0.015 0.1 0.04
