Commit message: Improved simulation of balancer

File: balboa/balancer.urdf (robot description, URDF)
Before this commit: robot physics, 3 links, 2 joints
Links:
- link baseLink: geometry collision box size=0.08 0.1 0.04; visual box size=0.04 0.04 0.04

Commit message: Fixed issue related to timestep size.

File: balboa/balancer.urdf (robot description, URDF)
Before this commit: robot physics, 3 links, 2 joints
Links:
- link baseLink: mass .3 -> .31; geometry collision box size=0.08 0.1 0.04; visual box size=0.04 0.04 0.04

Commit message: Accelerometer orientation seems ok now.

File: balboa/balancer.urdf (robot description, URDF)
Before this commit: robot physics, 3 links, 2 joints
Links:
- added link accelerometer, mass .01; visual box size=0.01 0.01 0.005
Joints:
- added joint accelerometer: type continuous, parent baseLink, child accelerometer, origin xyz=0 0 0 rpy=0 -1.5708 0, axis 0 0 -1

Commit message: Now with accelerometer offset, battery resistance, and better env configuration.
Signed-off-by: Charles Blouin <cha.blouin@gmail.com>

File: balboa/balancer.urdf (robot description, URDF)
Before this commit: robot physics, 4 links, 3 joints
Joints:
- joint accelerometer: origin xyz=0 0 0 rpy=0 -1.5708 0 -> xyz=0 -0.01 0.07 rpy=0 -1.5708 0
