Commit message: Working robot model. Needs to add motors.

File: walker_a/urdf/walker_a_0_5.urdf (robot description, URDF)
Before this commit: robot physics, 13 links, 12 joints
Links:
- removed link baseLink
- removed link leg_0_0
- removed link leg_0_1
- removed link leg_0_2
- removed link leg_1_0
- removed link leg_1_1
- removed link leg_1_2
- removed link leg_2_0
- removed link leg_2_1
- removed link leg_2_2
- removed link leg_3_0
- removed link leg_3_1
- removed link leg_3_2
- added link base_link, mass 40; collision mesh filename=body.obj scale=1 1 1; visual mesh filename=body.obj scale=1 1 1
- added link link_0_0, mass 2; collision mesh filename=leg_X_0.obj scale=1 1 1; visual mesh filename=leg_X_0.obj scale=1 1 1
- added link link_0_1, mass 2; collision mesh filename=leg_X_1.obj scale=1 1 1; visual mesh filename=leg_X_1.obj scale=1 1 1
- added link link_0_2, mass 2; collision mesh filename=leg_X_1.obj scale=1 1 1; visual mesh filename=leg_X_1.obj scale=1 1 1
- added link link_1_0, mass 2; collision mesh filename=leg_X_0.obj scale=1 1 1; visual mesh filename=leg_X_0.obj scale=1 1 1
- added link link_1_1, mass 2; collision mesh filename=leg_X_1.obj scale=1 1 1; visual mesh filename=leg_X_1.obj scale=1 1 1
- added link link_1_2, mass 2; collision mesh filename=leg_X_1.obj scale=1 1 1; visual mesh filename=leg_X_1.obj scale=1 1 1
- added link link_2_0, mass 2; collision mesh filename=leg_X_0.obj scale=1 1 1; visual mesh filename=leg_X_0.obj scale=1 1 1
- added link link_2_1, mass 2; collision mesh filename=leg_X_1.obj scale=1 1 1; visual mesh filename=leg_X_1.obj scale=1 1 1
- added link link_2_2, mass 2; collision mesh filename=leg_X_1.obj scale=1 1 1; visual mesh filename=leg_X_1.obj scale=1 1 1
- added link link_3_0, mass 2; collision mesh filename=leg_X_0.obj scale=1 1 1; visual mesh filename=leg_X_0.obj scale=1 1 1
- added link link_3_1, mass 2; collision mesh filename=leg_X_1.obj scale=1 1 1; visual mesh filename=leg_X_1.obj scale=1 1 1
- added link link_3_2, mass 2; collision mesh filename=leg_X_1.obj scale=1 1 1; visual mesh filename=leg_X_1.obj scale=1 1 1
Joints:
- joint joint_0_0: axis 1 0 0 -> 1, 0, 0; child leg_0_0 -> link_0_0; limit lower=-0.1 upper=0.1 effort=300 velocity=10 -> (none); origin xyz=0.35, -0.3, 0 rpy=0 0 0 -> xyz=0.35, -0.3, 0 rpy=0, 0, 0; parent baseLink -> base_link
- joint joint_0_1: axis 0 1 0 -> 0, 1, 0; child leg_0_1 -> link_0_1; limit lower=-0.1 upper=0.1 effort=300 velocity=10 -> (none); origin xyz=0.15, 0, 0 rpy=0 0 0 -> xyz=0.15, 0, 0; parent leg_0_0 -> link_0_0
- joint joint_0_2: axis 0 1 0 -> 0, 1, 0; child leg_0_2 -> link_0_2; limit lower=-0.1 upper=0.1 effort=300 velocity=10 -> (none); origin xyz=0, 0, -0.50 rpy=0 0 0 -> xyz=0, 0, -0.5; parent leg_0_1 -> link_0_1
- joint joint_1_0: axis 1 0 0 -> 1, 0, 0; child leg_1_0 -> link_1_0; limit lower=-0.1 upper=0.1 effort=300 velocity=10 -> (none); origin xyz=0.35, 0.3, 0 rpy=0 0 0 -> xyz=0.35, 0.3, 0 rpy=0, 0, 0; parent baseLink -> base_link
- joint joint_1_1: axis 0 1 0 -> 0, 1, 0; child leg_1_1 -> link_1_1; limit lower=-0.1 upper=0.1 effort=300 velocity=10 -> (none); origin xyz=0.15, 0, 0 rpy=0 0 0 -> xyz=0.15, 0, 0; parent leg_1_0 -> link_1_0
- joint joint_1_2: axis 0 1 0 -> 0, 1, 0; child leg_1_2 -> link_1_2; limit lower=-0.1 upper=0.1 effort=300 velocity=10 -> (none); origin xyz=0, 0, -0.50 rpy=0 0 0 -> xyz=0, 0, -0.5; parent leg_1_1 -> link_1_1
- joint joint_2_0: axis 1 0 0 -> 1, 0, 0; child leg_2_0 -> link_2_0; limit lower=-0.1 upper=0.1 effort=300 velocity=10 -> (none); origin xyz=-0.35, 0.3, 0 rpy=0 0 3.14159 -> xyz=-0.35, 0.3, 0 rpy=0, 0, 3.14159; parent baseLink -> base_link
- joint joint_2_1: axis 0 1 0 -> 0, 1, 0; child leg_2_1 -> link_2_1; limit lower=-0.1 upper=0.1 effort=300 velocity=10 -> (none); origin xyz=0.15, 0, 0 rpy=0 0 0 -> xyz=0.15, 0, 0; parent leg_2_0 -> link_2_0
- joint joint_2_2: axis 0 1 0 -> 0, 1, 0; child leg_2_2 -> link_2_2; limit lower=-0.1 upper=0.1 effort=300 velocity=10 -> (none); origin xyz=0, 0, -0.50 rpy=0 0 0 -> xyz=0, 0, -0.5; parent leg_2_1 -> link_2_1
- joint joint_3_0: axis 1 0 0 -> 1, 0, 0; child leg_3_0 -> link_3_0; limit lower=-0.1 upper=0.1 effort=300 velocity=10 -> (none); origin xyz=-0.35, -0.3, 0 rpy=0 0 3.14159 -> xyz=-0.35, -0.3, 0 rpy=0, 0, 3.14159; parent baseLink -> base_link
- joint joint_3_1: axis 0 1 0 -> 0, 1, 0; child leg_3_1 -> link_3_1; limit lower=-0.1 upper=0.1 effort=300 velocity=10 -> (none); origin xyz=0.15, 0, 0 rpy=0 0 0 -> xyz=0.15, 0, 0; parent leg_3_0 -> link_3_0
- joint joint_3_2: axis 0 1 0 -> 0, 1, 0; child leg_3_2 -> link_3_2; limit lower=-0.1 upper=0.1 effort=300 velocity=10 -> (none); origin xyz=0, 0, -0.50 rpy=0 0 0 -> xyz=0, 0, -0.5; parent leg_3_1 -> link_3_1
