Commit message: Can train really well with those parameters.

File: pendulum_a/urdf/pendulum_a.urdf (robot description, URDF)
Before this commit: robot physics, 3 links, 2 joints
Links:
- link arm_1: mass 0.01875 -> 0.0375

Commit message: before changing to sin and cos representation

File: pendulum_a/urdf/pendulum_a.urdf (robot description, URDF)
Before this commit: robot physics, 3 links, 2 joints
Links:
- link arm_1: geometry collision box size=0.025 0.0075 0.2; visual box size=0.025 0.0075 0.2
